Commit message: zed on turtlebot3

File: nano/catkin_ws/src/turtlebot3/turtlebot3_description/urdf/turtlebot3_burger.gazebo.xacro (robot description, xacro)
@@ -92,6 +92,7 @@
     </plugin>
   </gazebo>
-  <gazebo reference="base_scan">
-    <material>Gazebo/FlatBlack</material>
+  <gazebo reference="base_camera_right">
+    <material>Gazebo/SkyBlue</material>
+<!--
     <sensor type="ray" name="lds_lfcd_sensor">
       <pose>0 0 0 0 0 0</pose>
@@ -123,4 +124,113 @@
       </plugin>
     </sensor>
-  </gazebo>
+-->
+<!--  modify -->
+     <sensor name="camera_right(sensor)" type="camera">
+        <update_rate>20</update_rate>
+	<visualize>true</visualize>
+	<camera>
+          <horizontal_fov>1.047198</horizontal_fov>
+          <image>
+            <width>640</width>
+            <height>480</height>
+            <format>R8G8B8</format>
+          </image>
+          <clip>
+            <near>0.05</near>
+            <far>3</far>
+          </clip>
+          <noise>
+            <type>gaussian</type>
+            <!-- Noise is sampled independently per pixel on each frame.
+                 That pixel's noise value is added to each of its color
+                 channels, which at that point lie in the range [0,1]. -->
+            <mean>0.0</mean>
+            <stddev>0.007</stddev>
+          </noise>
+        </camera>
+        <plugin name="camera_right_plugin" filename="libgazebo_ros_camera.so">
+          <alwaysOn>true</alwaysOn>
+          <updateRate>0.0</updateRate>
+          <cameraName>camera_right</cameraName>
+          <imageTopicName>image_raw</imageTopicName>
+          <cameraInfoTopicName>camera_info</cameraInfoTopicName>
+          <frameName>camera_link</frameName>
+          <hackBaseline>0.0</hackBaseline>
+          <distortionK1>0.0</distortionK1>
+          <distortionK2>0.0</distortionK2>
+          <distortionK3>0.0</distortionK3>
+          <distortionT1>0.0</distortionT1>
+          <distortionT2>0.0</distortionT2>
+        </plugin>
+      </sensor>
+<!-- modify -->
+  </gazebo>
+<!-- modify-->
+  <gazebo reference="base_camera_left">
+    <material>Gazebo/White</material>
+      <sensor name="camera_left(sensor)" type="camera">
+        <update_rate>20</update_rate>
+        <camera name="left_crazy_camera">
+          <pose> 0 0 0 0 0 0 </pose>
+          <horizontal_fov>1.047198</horizontal_fov>
+          <image>
+            <width>640</width>
+            <height>480</height>
+            <format>R8G8B8</format>
+          </image>
+          <clip>
+            <near>0.05</near>
+            <far>3</far>
+          </clip>
+          <noise>
+            <type>gaussian</type>
+            <mean>0.0</mean>
+            <stddev>0.007</stddev>
+          </noise>
+        </camera>
+        <plugin name="camera_left_plugin" filename="libgazebo_ros_camera.so">
+          <alwaysOn>true</alwaysOn>
+          <updateRate>0.0</updateRate>
+          <cameraName>camera_left</cameraName>
+          <imageTopicName>image_raw</imageTopicName>
+          <cameraInfoTopicName>camera_info</cameraInfoTopicName>
+          <frameName>camera_link</frameName>
+          <hackBaseline>0.0</hackBaseline>
+          <distortionK1>0.0</distortionK1>
+          <distortionK2>0.0</distortionK2>
+          <distortionK3>0.0</distortionK3>
+          <distortionT1>0.0</distortionT1>
+          <distortionT2>0.0</distortionT2>
+        </plugin>
+      </sensor>
+  </gazebo>
+  <gazebo reference="base_camera_depth">
+    <material>Gazebo/Green</material>
+    <sensor name="camera_depth(sensor)" type="depth">
+      <update_rate>20</update_rate>
+      <camera>
+      <horizontal_fov>1.047198</horizontal_fov>
+        <image>
+          <width>16</width>
+          <height>12</height>
+          <format>R8G8B8</format>
+        </image>
+        <clip>
+          <near>0.05</near>
+          <far>3</far>
+        </clip>
+      </camera>
+      <plugin name="camera_depth_plugin" filename="libgazebo_ros_depth_camera.so">
+        <cameraName>camera_depth</cameraName>
+        <alwaysOn>true</alwaysOn>
+        <updateRate>0</updateRate>
+        <imageTopicName>depth_camera/image</imageTopicName>
+        <depthImageTopicName>depth_camera/depth_image</depthImageTopicName>
+        <cameraInfoTopicName>depth_camera/camera_info</cameraInfoTopicName>
+        <depthCameraInfoTopicName>depth_camera/depth_camera_info</depthCameraInfoTopicName>
+        <frameName>camera_link</frameName>
+      </plugin>
+    </sensor>
+  </gazebo>
+<!-- modify-->
 </robot>

File: nano/catkin_ws/src/turtlebot3/turtlebot3_description/urdf/turtlebot3_burger.urdf.xacro (robot description, xacro)
@@ -113,16 +113,73 @@
   </joint>
   <link name="imu_link"/>
-  <joint name="scan_joint" type="fixed">
+<!--             right camera                    -->
+  <joint name="camera_right_joint" type="fixed">
     <parent link="base_link"/>
-    <child link="base_scan"/>
-    <origin xyz="-0.032 0 0.172" rpy="0 0 0"/>
+    <child link="base_camera_right"/>
+    <origin xyz="-0.032 -0.03 0.172" rpy="0 0 0"/>
   </joint>
-  <link name="base_scan">
+  <link name="base_camera_right">
     <visual>
-      <origin xyz="0 0 0.0" rpy="0 0 0"/>
+      <origin xyz="0 0 0" rpy="0 0 0"/>
       <geometry>
-        <mesh filename="package://turtlebot3_description/meshes/sensors/lds.stl" scale="0.001 0.001 0.001"/>
+        <mesh filename="package://turtlebot3_description/meshes/sensors/lds.stl" scale="0.0003 0.0003 0.0003"/>
       </geometry>
-      <material name="dark"/>
+      <material name="blue"/>
+    </visual>
+    <collision>
+      <origin xyz="0.015 0 -0.0065" rpy="0 0 0"/>
+      <geometry>
+        <cylinder length="0.0315" radius="0.055"/>
+      </geometry>
+    </collision>
+    <inertial>
+      <mass value="0.114" />
+      <origin xyz="0 0 0" />
+      <inertia ixx="0.001" ixy="0.0" ixz="0.0"
+               iyy="0.001" iyz="0.0"
+               izz="0.001" />
+    </inertial>
+  </link>
+<!--             left camera            -->
+  <joint name="camera_left_joint" type="fixed">
+    <parent link="base_link"/>
+    <child link="base_camera_left"/>
+    <origin xyz="-0.032 0.02 0.172" rpy="0 0 0"/>
+  </joint>
+  <link name="base_camera_left">
+    <visual>
+      <origin xyz="0 0 0" rpy="0 0 0"/>
+      <geometry>
+        <mesh filename="package://turtlebot3_description/meshes/sensors/lds.stl" scale="0.0003 0.0003 0.0003"/>
+      </geometry>
+      <material name="white"/>
+    </visual>
+    <collision>
+      <origin xyz="0.015 0 -0.0065" rpy="0 0 0"/>
+      <geometry>
+        <cylinder length="0.0315" radius="0.055"/>
+      </geometry>
+    </collision>
+    <inertial>
+      <mass value="0.114" />
+      <origin xyz="0 0 0" />
+      <inertia ixx="0.001" ixy="0.0" ixz="0.0"
+               iyy="0.001" iyz="0.0"
+               izz="0.001" />
+    </inertial>
+  </link>
+<!-- depth camera-->
+  <joint name="camera_depth_joint" type="fixed">
+    <parent link="base_link"/>
+    <child link="base_camera_depth"/>
+    <origin xyz="-0.032 -0.005 0.172" rpy="0 0 0"/>
+  </joint>
+  <link name="base_camera_depth">
+    <visual>
+      <origin xyz="0 0 0" rpy="0 0 0"/>
+      <geometry>
+        <mesh filename="package://turtlebot3_description/meshes/sensors/lds.stl" scale="0.0002 0.0002 0.0002"/>
+      </geometry>
+      <material name="red"/>
     </visual>
     <collision>
