Commit message: zed listener (transform to distance matrix)

File: nano/catkin_ws/src/turtlebot3/turtlebot3_description/urdf/fake_turtlebot3_burger.gazebo.xacro (robot description, xacro)
@@ -97,13 +97,11 @@
       <visualize>true</visualize>
       <camera>
-        <horizontal_fov>2.094396</horizontal_fov>  <!--<horizontal_fov>1.047198</horizontal_fov> -->
+	<pose>0.01 0 0 0 0 0</pose>
+        <horizontal_fov>2.094396</horizontal_fov> <!--<horizontal_fov>1.047198</horizontal_fov> -->
         <image>
-          <width>640</width>
-          <height>480</height>
+          <width>16</width>
+          <height>12</height>
           <format>R8G8B8</format>
         </image>
-	<depth_camera>
-	    <output>depthImage</output>
-	</depth_camera>
         <clip>
           <near>0.05</near>
@@ -118,5 +116,5 @@
         <depthImageTopicName>depth_camera/depth_image</depthImageTopicName>
         <cameraInfoTopicName>depth_camera/camera_info</cameraInfoTopicName>
-        <ImageInfoTopicName>depth_camera_image</ImageInfoTopicName>
+        <depthCameraInfoTopicName>depth_camera/depth_camera_info</depthCameraInfoTopicName>
         <frameName>camera_link</frameName>
       </plugin>

File: nano/catkin_ws/src/turtlebot3/turtlebot3_description/urdf/fake_turtlebot3_burger.urdf.xacro (robot description, xacro)
@@ -121,5 +121,5 @@
   <link name="base_camera_depth">
     <visual>
-      <origin xyz="0 0 0" rpy="1.57 0 1.57"/>
+      <origin xyz="0 0 0" rpy="1.5707963 0 1.5707963"/>
       <geometry>
     <!--    <mesh filename="package://turtlebot3_description/meshes/sensors/lds.stl" scale="0.0002 0.0002 0.0002"/> -->
