Commit message: fit to pbot meshes

File: alice/alice-ros/pairbot/src/pairbot/pb_description/urdf/pairbot.xacro (robot description, xacro)
@@ -3,33 +3,32 @@
 <robot name="pairbot" xmlns:xacro="http://www.ros.org/wiki/xacro">
     <!-- Constants for robot dimensions -->
-    <xacro:property name="PI" value="3.1415"/>
-    <xacro:property name="M_PI" value="3.1415"/>
-    <xacro:property name="width" value="0"/>
+    <xacro:property name="PI" value="3.1415926"/>
     <!-- Square dimensions (width x width) of beams  0.1-->
-    <xacro:property name="camera_link" value="0.05"/>
-    <xacro:property name="axel_offset" value="0.05"/>
-    <xacro:property name="base_link_size_x" value="2.56"/> <!--was 0.397-->
-    <xacro:property name="base_link_size_y" value="3.85"/>  <!--was 0.1789-->
-    <xacro:property name="base_link_size_z"
-                    value="${2*wheel_radius-ground_clearance}"/>   <!-- old 0.102 is double radius without ground_clearance 0.07683 -->
-    <xacro:property name="big_wheel_radius" value="0.8"/>   <!--was 0.09-->
-    <xacro:property name="small_wheel_radius" value="${big_wheel_radius*0.3}"/>   <!--was 0.09-->
-    <xacro:property name="flipper_wheel_radius" value="${small_wheel_radius*0.6}"/>
-    <xacro:property name="flipper_wheel_slope" value="0.04"/>
-    <xacro:property name="flipper_wheel_bias" value="${0.8*small_wheel_radius}"/>
-    <xacro:property name="ground_clearance" value="0.02517"/>   <!--old 0.05 0.02517-->
-    <xacro:property name="wheel_length" value="${0.22*scale}"/>
-    <xacro:property name="wheel_mass" value="0.1"/>
-    <xacro:property name="scale" value="0.1"/>
+    <xacro:property name="base_length" value="0.6"/> <!--was 0.397-->
+    <xacro:property name="base_width"  value="0.42"/>  <!--was 0.1789-->
+    <xacro:property name="base_height" value="0.18"/>
+    <xacro:property name="gear_length" value="0.54"/>
+    <xacro:property name="gear_width"  value="0.136"/> <!-- = 0.20-0.064 -->
+    <xacro:property name="gear_height" value="0.16"/>
+    <xacro:property name="big_wheel_radius" value="0.05"/>   <!--was 0.09-->
+    <xacro:property name="big_wheel_length" value="0.028"/>
+    <xacro:property name="flipper_length" value="0.42"/>
+    <xacro:property name="flipper_width" value="0.10"/>
+    <xacro:property name="flipper_height" value="0.1578"/>
+    <xacro:property name="flipper_wheel_radius" value="0.03"/>
+    <xacro:property name="flipper_wheel_length" value="0.017"/>
+    <xacro:property name="flipper_wheel_distance" value="0.065"/>
+    <!-- <xacro:property name="ground_clearance" value="0.02517"/>  old 0.05 0.02517-->
+    <xacro:property name="scale" value="1"/>
     <xacro:property name="prefix" value="pairbot"/>
-    <xacro:property name="base_mass" value="100"/> <!--100-->
-    <xacro:property name="flipper_mass" value="77.5"/> <!--77.5-->
-    <xacro:property name="big_wheel_mass" value="30"/>
-    <xacro:property name="small_wheel_mass" value="10"/>
+    <xacro:property name="base_mass" value="40.0"/> <!--100-->
+    <xacro:property name="flipper_mass" value="2.5"/> <!--77.5-->
+    <xacro:property name="big_wheel_mass" value="0.1"/>
+    <xacro:property name="small_wheel_mass" value="0.1"/>
     <xacro:include filename="$(find pb_description)/urdf/pairbot.gazebo"/>
     <xacro:include filename="$(find pb_description)/urdf/materials.xacro"/>
     <!-- <xacro:include filename="$(find husky_description)/urdf/accessories/sick_lms1xx_mount.urdf.xacro"/> -->
     <xacro:macro name="collision_macro"
-                 params="mesh_name x y z roll pitch yaw scale">
+                 params="mesh_name x y z roll pitch yaw scale:=${scale}">
         <collision>
             <origin xyz="${x} ${y} ${z}" rpy="${roll} ${pitch} ${yaw}"/>
@@ -89,18 +88,12 @@
     </xacro:macro>
     <xacro:macro name="wheel"
-                 params="mesh_name material name_link x y z roll pitch yaw radius wheel_length mass parent">
+                 params="mesh_name material name_link x y z roll pitch yaw radius wheel_length mass parent direction:=1">
         <link name="${name_link}">
-            <xacro:visual_macro mesh_name="${mesh_name}" x="0" y="0" z="0" roll="1.57" pitch="0" yaw="0"
-                                material="${material}" scale="${0.030*radius*scale}"/>
-            <!--<visual>
-                <origin xyz="0 0 0" rpy="0 0 0"/>
+            <xacro:visual_macro mesh_name="${mesh_name}" x="0" y="0" z="0" roll="0" pitch="0" yaw="0"
+                                material="${material}" scale="${scale}"/>
+            <collision>
+                <origin xyz="0 0 0" rpy="${PI/2} 0 0"/>
                 <geometry>
-                    <cylinder radius='${radius*scale}' length="${wheel_length*scale}"/>
-                 </geometry>
-            </visual>-->
-            <collision>
-                <origin xyz="0 0 0" rpy="0 0 0"/>
-                <geometry>
-                    <cylinder radius='${radius*scale}' length="${wheel_length*scale}"/>
+                	<cylinder radius="${radius*scale}" length="${wheel_length*scale}"/>
                 </geometry>
             </collision>
@@ -113,5 +106,5 @@
             <child link="${name_link}"/>
             <origin xyz="${x} ${y} ${z}" rpy="${roll} ${pitch} ${yaw}"/>
-            <axis xyz="0 0 1"/>
+            <axis xyz="0 ${direction} 0"/>
             <limit velocity="20" effort="100"/>
         </joint>
@@ -127,166 +120,112 @@
         </transmission>
     </xacro:macro>
-    <xacro:link_macro name_link="base_link" x="0" y="0" z="0" roll="0" pitch="0" yaw="0" mesh_name="Base2.dae" mass="${base_mass}" material="orange"
+    <link name="base_link">
+        <xacro:visual_macro mesh_name="mainbody.stl" x="0" y="0" z="0" roll="0" pitch="0" yaw="0"
+                                material="orange" scale="${scale}"/>
+        <xacro:visual_macro mesh_name="left_gears.stl" x="0" y="${base_width/2}" z="0" roll="0" pitch="0" yaw="0"
+                                material="grey" scale="${scale}"/>
+        <xacro:visual_macro mesh_name="right_gears.stl" x="0" y="${-1*base_width/2}" z="0" roll="0" pitch="0" yaw="0"
+                                material="grey" scale="${scale}"/>
+        <xacro:collision_macro mesh_name="mainbody.stl" x="0" y="0" z="0" roll="0" pitch="0" yaw="0"
+                                   scale="${scale}"/>
+        <xacro:inertial_macro x="0" y="0" z="0"
+                                  roll="0" pitch="0" yaw="0" mass="${base_mass}"
+                                  ixx="1" ixy="0" ixz="0" iyy="1" iyz="0" izz="1"/>
+    </link>
+    <xacro:wheel name_link="right_front_base_link_wheel" mesh_name="right_tire.stl" material="grey"
+                 x="${(big_wheel_radius*2+0.01)*scale}" y="${-1*base_width/2*scale}" z="${(big_wheel_radius-0.04)*scale}" roll="0" pitch="0" yaw="0"
+                 radius="${big_wheel_radius}" wheel_length="${big_wheel_length}" mass="${big_wheel_mass}" parent="base_link"/>
+    <xacro:wheel name_link="right_middle_base_link_wheel"  mesh_name="right_tire.stl" material="grey"
+                 x="0" y="${-1*base_width/2*scale}" z="${(big_wheel_radius-0.04)*scale}" roll="0" pitch="0" yaw="0"
+                 radius="${big_wheel_radius}" wheel_length="${big_wheel_length}" mass="${big_wheel_mass}" parent="base_link"/>
+    <xacro:wheel name_link="right_rear_base_link_wheel" mesh_name="right_tire.stl" material="grey"
+                 x="${-1*(big_wheel_radius*2+0.01)*scale}" y="${-1*base_width/2*scale}" z="${(big_wheel_radius-0.04)*scale}" roll="0" pitch="0" yaw="0"
+                 radius="${big_wheel_radius}" wheel_length="${big_wheel_length}" mass="${big_wheel_mass}" parent="base_link"/>
+    <xacro:wheel name_link="left_front_base_link_wheel" mesh_name="left_tire.stl" material="grey"
+                 x="${(big_wheel_radius*2+0.01)*scale}" y="${base_width/2*scale}" z="${(big_wheel_radius-0.04)*scale}" roll="0" pitch="0" yaw="0"
+                 radius="${big_wheel_radius}" wheel_length="${big_wheel_length}" mass="${big_wheel_mass}" parent="base_link"/>
+    <xacro:wheel name_link="left_middle_base_link_wheel" mesh_name="left_tire.stl" material="grey"
+                 x="0" y="${base_width/2*scale}" z="${(big_wheel_radius-0.04)*scale}" roll="0" pitch="0" yaw="0"
+                radius="${big_wheel_radius}" wheel_length="${big_wheel_length}" mass="${big_wheel_mass}" parent="base_link"/>
+    <xacro:wheel name_link="left_rear_base_link_wheel" mesh_name="left_tire.stl" material="grey"
+                 x="${-1*(big_wheel_radius*2+0.01)*scale}" y="${base_width/2*scale}" z="${(big_wheel_radius-0.04)*scale}" roll="0" pitch="0" yaw="0"
+                 radius="${big_wheel_radius}" wheel_length="${big_wheel_length}" mass="${big_wheel_mass}" parent="base_link"/>
+<!-- y=3.4 x=0.3--> <!--for flipper: x: left/right y: up/down-->
+    <xacro:macro name="right_flipper_asm"
+        params="loc jx jy jz roll pitch yaw direction:=1">
+        <xacro:link_macro name_link="${loc}_flipper" x="0" y="0" z="0" roll="0" pitch="0" yaw="0" mesh_name="right_front_flipper.stl"  mass="${flipper_mass}" material="grey"
                       scale="${scale}" ixx="1" ixy="0.0" ixz="0.0" iyy="1" iyz="0.000" izz="1"/>
-    <!--front flipper-->
-    <xacro:link_macro name_link="right_front_flipper" x="0" y="0" z="0" roll="0" pitch="0" yaw="0" mesh_name="RightFrontFlipper.dae" mass="${flipper_mass}" material="grey"
-                      scale="${scale}" ixx="1" ixy="0.0" ixz="0.0" iyy="1" iyz="0.000" izz="1"/>
-    <xacro:joint_macro joint_name="joint_right_front_flipper" type="continuous" parent="base_link" child="right_front_flipper"
-                       x="${1.86*scale}" y="${-2.2*scale}" z="${-0.25*scale}" roll="${-PI*0.5}" pitch="0" yaw="${-PI/2}" axis="1 0 0" />
-    <!-- <xacro:joint_macro joint_name="joint_right_front_flipper" type="revolute" parent="base_link" child="right_front_flipper"
-                       x="${1.86*scale}" y="${-3.0*scale}" z="${-0.25*scale}" roll="${-PI*0.5}" pitch="0" yaw="${-PI/2}" axis="1 0 0" /> -->
-    <xacro:link_macro name_link="left_front_flipper" x="0" y="0" z="0" roll="0" pitch="0" yaw="0" mesh_name="LeftFrontFlipper.dae" mass="${flipper_mass}" material="grey"
-                      scale="${scale}" ixx="1" ixy="0.0" ixz="0.0" iyy="1" iyz="0.000" izz="1"/>
-    <xacro:joint_macro joint_name="joint_left_front_flipper" type="continuous" parent="base_link" child="left_front_flipper"
-                       x="${1.86*scale}" y="${2.2*scale}" z="${-0.25*scale}" roll="${-PI*0.5}" pitch="0" yaw="${-PI/2}" axis="1 0 0"/>
-    <!-- <xacro:joint_macro joint_name="joint_left_front_flipper" type="continuous" parent="base_link" child="left_front_flipper"
-                       x="${1.86*scale}" y="${2.2*scale}" z="${-0.25*scale}" roll="${-PI*0.5}" pitch="0" yaw="${-PI/2}" axis="1 0 0"/> -->
-    <!--rear flipper-->
-    <xacro:link_macro name_link="right_rear_flipper" x="0" y="0" z="0" roll="0" pitch="0" yaw="0" mesh_name="RightRearFlipper.dae" mass="${flipper_mass}" material="grey"
-                      scale="${scale}" ixx="1" ixy="0.0" ixz="0.0" iyy="1" iyz="0.000" izz="1"/>
-    <xacro:joint_macro joint_name="joint_right_rear_flipper" type="continuous" parent="base_link" child="right_rear_flipper"
-                       x="${-1.86*scale}" y="${-2.2*scale}" z="${-0.25*scale}" roll="${PI*0.5}" pitch="0" yaw="${-PI/2}" axis="-1 0 0" />
-    <xacro:link_macro name_link="left_rear_flipper" x="0" y="0" z="0" roll="0" pitch="0" yaw="0" mesh_name="LeftRearFlipper.dae" mass="${flipper_mass}" material="grey"
-                      scale="${scale}" ixx="1" ixy="0.0" ixz="0.0" iyy="1" iyz="0.000" izz="1"/>
-    <xacro:joint_macro joint_name="joint_left_rear_flipper" type="continuous" parent="base_link" child="left_rear_flipper"
-                       x="${-1.86*scale}" y="${2.2*scale}" z="${-0.25*scale}" roll="${PI*0.5}" pitch="0" yaw="${-PI/2}" axis="-1 0 0"/>
-    <xacro:wheel name_link="right_front_base_link_wheel" mesh_name="right_tire.stl" material="grey"
-                 x="${1.86*scale}" y="${-2.75*scale}" z="${-0.25*scale}" roll="0" pitch="${PI*0.5}" yaw="${PI/2}"
-                 radius="${big_wheel_radius}" wheel_length="${wheel_length}" mass="${big_wheel_mass}" parent="base_link"/>
-    <xacro:wheel name_link="left_front_base_link_wheel" mesh_name="left_tire.stl" material="grey"
-                 x="${1.86*scale}" y="${2.75*scale}" z="${-0.25*scale}" roll="0" pitch="${PI*0.5}" yaw="${PI/2}"
-                 radius="${big_wheel_radius}" wheel_length="${wheel_length}" mass="${big_wheel_mass}" parent="base_link"/>
-    <xacro:wheel name_link="right_rear_base_link_wheel" mesh_name="right_tire.stl" material="grey"
-                 x="${-1.86*scale}" y="${-2.75*scale}" z="${-0.25*scale}" roll="0" pitch="${PI*0.5}" yaw="${PI/2}"
-                 radius="${big_wheel_radius}" wheel_length="${wheel_length}" mass="${big_wheel_mass}" parent="base_link"/>
-    <xacro:wheel name_link="left_rear_base_link_wheel" mesh_name="left_tire.stl" material="grey"
-                 x="${-1.86*scale}" y="${2.75*scale}" z="${-0.25*scale}" roll="0" pitch="${PI*0.5}" yaw="${PI/2}"
-                 radius="${big_wheel_radius}" wheel_length="${wheel_length}" mass="${big_wheel_mass}" parent="base_link"/>
-    <xacro:wheel name_link="right_middle_base_link_wheel"  mesh_name="right_tire.stl" material="grey"
-                x="0" y="${-2.75*scale}" z="${-0.25*scale}" roll="0" pitch="${PI*0.5}" yaw="${PI/2}"
-                radius="${big_wheel_radius}" wheel_length="${wheel_length}" mass="${big_wheel_mass}" parent="base_link"/>
-    <xacro:wheel name_link="left_middle_base_link_wheel" mesh_name="left_tire.stl" material="grey"
-                 x="0" y="${2.75*scale}" z="${-0.25*scale}" roll="0" pitch="${PI*0.5}" yaw="${PI/2}"
-                radius="${big_wheel_radius}" wheel_length="${wheel_length}" mass="${big_wheel_mass}" parent="base_link"/>
-<!-- y=3.4 x=0.3--> <!--for flipper: x: left/right y: up/down-->
-    <!-- right front flipper -->
-    <xacro:wheel name_link="right_front_flipper_wheel" mesh_name="right_tire.stl" material="grey"
-                 x="${0.5*scale}" y="${flipper_wheel_bias*scale}" z="${3.4*scale}"
-                 roll="0" pitch="${PI*0.5}" yaw="${PI}"
-                 radius="${small_wheel_radius}" wheel_length="${wheel_length}" mass="${small_wheel_mass}" parent="right_front_flipper"/>
-    <xacro:wheel name_link="right_front_flipper_middle_wheel_1" mesh_name="right_tire.stl" material="grey"
-                 x="${0.5*scale}" y="${1*flipper_wheel_slope*scale+flipper_wheel_bias*scale}" z="${3.4*scale-2*small_wheel_radius*scale}"
-                 roll="0" pitch="${PI*0.5}" yaw="${PI}"
-                 radius="${small_wheel_radius}" wheel_length="${wheel_length}" mass="${small_wheel_mass}" parent="right_front_flipper"/>
-    <xacro:wheel name_link="right_front_flipper_middle_wheel_2" mesh_name="right_tire.stl" material="grey"
-                 x="${0.5*scale}" y="${2*flipper_wheel_slope*scale+flipper_wheel_bias*scale}" z="${3.4*scale-4*small_wheel_radius*scale}"
-                 roll="0" pitch="${PI*0.5}" yaw="${PI}"
-                 radius="${small_wheel_radius}" wheel_length="${wheel_length}" mass="${small_wheel_mass}" parent="right_front_flipper"/>
-    <xacro:wheel name_link="right_front_flipper_middle_wheel_3" mesh_name="right_tire.stl" material="grey"
-                 x="${0.5*scale}" y="${3*flipper_wheel_slope*scale+flipper_wheel_bias*scale}" z="${3.4*scale-6*small_wheel_radius*scale}"
-                 roll="0" pitch="${PI*0.5}" yaw="${PI}"
-                 radius="${small_wheel_radius}" wheel_length="${wheel_length}" mass="${small_wheel_mass}" parent="right_front_flipper"/>
-    <xacro:wheel name_link="right_front_flipper_middle_wheel_4" mesh_name="right_tire.stl" material="grey"
-                 x="${0.5*scale}" y="${4*flipper_wheel_slope*scale+flipper_wheel_bias*scale}" z="${3.4*scale-8*small_wheel_radius*scale}"
-                 roll="0" pitch="${PI*0.5}" yaw="${PI}"
-                 radius="${small_wheel_radius}" wheel_length="${wheel_length}" mass="${small_wheel_mass}" parent="right_front_flipper"/>
-    <xacro:wheel name_link="right_front_flipper_middle_wheel_5" mesh_name="right_tire.stl" material="grey"
-                 x="${0.5*scale}" y="${5*flipper_wheel_slope*scale+flipper_wheel_bias*scale}" z="${3.4*scale-10*small_wheel_radius*scale}"
-                 roll="0" pitch="${PI*0.5}" yaw="${PI}"
-                 radius="${small_wheel_radius}" wheel_length="${wheel_length}" mass="${small_wheel_mass}" parent="right_front_flipper"/>
-    <!-- left front flipper -->
-    <xacro:wheel name_link="left_front_flipper_wheel"  mesh_name="left_tire.stl" material="grey"
-                 x="${-0.5*scale}" y="${flipper_wheel_bias*scale}" z="${3.4*scale}"
-                 roll="0" pitch="${PI*0.5}" yaw="${PI}"
-                 radius="${small_wheel_radius}" wheel_length="${wheel_length}" mass="${small_wheel_mass}" parent="left_front_flipper"/>
-    <xacro:wheel name_link="left_front_flipper_middle_wheel_1" mesh_name="left_tire.stl" material="grey"
-                 x="${-0.5*scale}" y="${1*flipper_wheel_slope*scale+flipper_wheel_bias*scale}" z="${3.4*scale-2*small_wheel_radius*scale}"
-                 roll="0" pitch="${PI*0.5}" yaw="${PI}"
-                 radius="${small_wheel_radius}" wheel_length="${wheel_length}" mass="${small_wheel_mass}" parent="left_front_flipper"/>
-    <xacro:wheel name_link="left_front_flipper_middle_wheel_2" mesh_name="left_tire.stl" material="grey"
-                 x="${-0.5*scale}" y="${2*flipper_wheel_slope*scale+flipper_wheel_bias*scale}" z="${3.4*scale-4*small_wheel_radius*scale}"
-                 roll="0" pitch="${PI*0.5}" yaw="${PI}"
-                 radius="${small_wheel_radius}" wheel_length="${wheel_length}" mass="${small_wheel_mass}" parent="left_front_flipper"/>
-    <xacro:wheel name_link="left_front_flipper_middle_wheel_3" mesh_name="left_tire.stl" material="grey"
-                 x="${-0.5*scale}" y="${3*flipper_wheel_slope*scale+flipper_wheel_bias*scale}" z="${3.4*scale-6*small_wheel_radius*scale}"
-                 roll="0" pitch="${PI*0.5}" yaw="${PI}"
-                 radius="${small_wheel_radius}" wheel_length="${wheel_length}" mass="${small_wheel_mass}" parent="left_front_flipper"/>
-    <xacro:wheel name_link="left_front_flipper_middle_wheel_4" mesh_name="left_tire.stl" material="grey"
-                 x="${-0.5*scale}" y="${4*flipper_wheel_slope*scale+flipper_wheel_bias*scale}" z="${3.4*scale-8*small_wheel_radius*scale}"
-                 roll="0" pitch="${PI*0.5}" yaw="${PI}"
-                 radius="${small_wheel_radius}" wheel_length="${wheel_length}" mass="${small_wheel_mass}" parent="left_front_flipper"/>
-    <xacro:wheel name_link="left_front_flipper_middle_wheel_5" mesh_name="left_tire.stl" material="grey"
-                 x="${-0.5*scale}" y="${5*flipper_wheel_slope*scale+flipper_wheel_bias*scale}" z="${3.4*scale-10*small_wheel_radius*scale}"
-                 roll="0" pitch="${PI*0.5}" yaw="${PI}"
-                 radius="${small_wheel_radius}" wheel_length="${wheel_length}" mass="${small_wheel_mass}" parent="left_front_flipper"/>
-    <!-- right rear flipper -->
-    <xacro:wheel name_link="right_rear_flipper_wheel" mesh_name="right_tire.stl" material="grey"
-                 x="${0.5*scale}" y="${-flipper_wheel_bias*scale}" z="${3.4*scale}"
-                 roll="0" pitch="${PI*0.5}" yaw="${PI}"
-                 radius="${small_wheel_radius}" wheel_length="${wheel_length}" mass="${small_wheel_mass}" parent="right_rear_flipper"/>
-    <xacro:wheel name_link="right_rear_flipper_middle_wheel_1" mesh_name="right_tire.stl" material="grey"
-                 x="${0.5*scale}" y="${-1*flipper_wheel_slope*scale-flipper_wheel_bias*scale}" z="${3.4*scale-2*small_wheel_radius*scale}"
-                 roll="0" pitch="${PI*0.5}" yaw="${PI}"
-                 radius="${small_wheel_radius}" wheel_length="${wheel_length}" mass="${small_wheel_mass}" parent="right_rear_flipper"/>
-    <xacro:wheel name_link="right_rear_flipper_middle_wheel_2" mesh_name="right_tire.stl" material="grey"
-                 x="${0.5*scale}" y="${-2*flipper_wheel_slope*scale-flipper_wheel_bias*scale}" z="${3.4*scale-4*small_wheel_radius*scale}"
-                 roll="0" pitch="${PI*0.5}" yaw="${PI}"
-                 radius="${small_wheel_radius}" wheel_length="${wheel_length}" mass="${small_wheel_mass}" parent="right_rear_flipper"/>
-    <xacro:wheel name_link="right_rear_flipper_middle_wheel_3"  mesh_name="right_tire.stl" material="grey"
-                 x="${0.5*scale}" y="${-3*flipper_wheel_slope*scale-flipper_wheel_bias*scale}" z="${3.4*scale-6*small_wheel_radius*scale}"
-                 roll="0" pitch="${PI*0.5}" yaw="${PI}"
-                 radius="${small_wheel_radius}" wheel_length="${wheel_length}" mass="${small_wheel_mass}" parent="right_rear_flipper"/>
-    <xacro:wheel name_link="right_rear_flipper_middle_wheel_4" mesh_name="right_tire.stl" material="grey"
-                 x="${0.5*scale}" y="${-4*flipper_wheel_slope*scale-flipper_wheel_bias*scale}" z="${3.4*scale-8*small_wheel_radius*scale}"
-                 roll="0" pitch="${PI*0.5}" yaw="${PI}"
-                 radius="${small_wheel_radius}" wheel_length="${wheel_length}" mass="${small_wheel_mass}" parent="right_rear_flipper"/>
-    <xacro:wheel name_link="right_rear_flipper_middle_wheel_5" mesh_name="right_tire.stl" material="grey"
-                 x="${0.5*scale}" y="${-5*flipper_wheel_slope*scale-flipper_wheel_bias*scale}" z="${3.4*scale-10*small_wheel_radius*scale}"
-                 roll="0" pitch="${PI*0.5}" yaw="${PI}"
-                 radius="${small_wheel_radius}" wheel_length="${wheel_length}" mass="${small_wheel_mass}" parent="right_rear_flipper"/>
-    <!-- left rear flipper -->
-    <xacro:wheel name_link="left_rear_flipper_wheel"  mesh_name="left_tire.stl" material="grey"
-                 x="${-0.5*scale}" y="${-flipper_wheel_bias*scale}" z="${3.4*scale}"
-                 roll="0" pitch="${PI*0.5}" yaw="${PI}"
-                 radius="${small_wheel_radius}" wheel_length="${wheel_length}" mass="${small_wheel_mass}" parent="left_rear_flipper"/>
-    <xacro:wheel name_link="left_rear_flipper_middle_wheel_1" mesh_name="left_tire.stl" material="grey"
-                 x="${-0.5*scale}" y="${-1*flipper_wheel_slope*scale-flipper_wheel_bias*scale}" z="${3.4*scale-2*small_wheel_radius*scale}"
-                 roll="0" pitch="${PI*0.5}" yaw="${PI}"
-                 radius="${small_wheel_radius}" wheel_length="${wheel_length}" mass="${small_wheel_mass}" parent="left_rear_flipper"/>
-    <xacro:wheel name_link="left_rear_flipper_middle_wheel_2" mesh_name="left_tire.stl" material="grey"
-                 x="${-0.5*scale}" y="${-2*flipper_wheel_slope*scale-flipper_wheel_bias*scale}" z="${3.4*scale-4*small_wheel_radius*scale}"
-                 roll="0" pitch="${PI*0.5}" yaw="${PI}"
-                 radius="${small_wheel_radius}" wheel_length="${wheel_length}" mass="${small_wheel_mass}" parent="left_rear_flipper"/>
-    <xacro:wheel name_link="left_rear_flipper_middle_wheel_3" mesh_name="left_tire.stl" material="grey"
-                 x="${-0.5*scale}" y="${-3*flipper_wheel_slope*scale-flipper_wheel_bias*scale}" z="${3.4*scale-6*small_wheel_radius*scale}"
-                 roll="0" pitch="${PI*0.5}" yaw="${PI}"
-                 radius="${small_wheel_radius}" wheel_length="${wheel_length}" mass="${small_wheel_mass}" parent="left_rear_flipper"/>
-    <xacro:wheel name_link="left_rear_flipper_middle_wheel_4" mesh_name="left_tire.stl" material="grey"
-                 x="${-0.5*scale}" y="${-4*flipper_wheel_slope*scale-flipper_wheel_bias*scale}" z="${3.4*scale-8*small_wheel_radius*scale}"
-                 roll="0" pitch="${PI*0.5}" yaw="${PI}"
-                 radius="${small_wheel_radius}" wheel_length="${wheel_length}" mass="${small_wheel_mass}" parent="left_rear_flipper"/>
-    <xacro:wheel name_link="left_rear_flipper_middle_wheel_5" mesh_name="left_tire.stl" material="grey"
-                 x="${-0.5*scale}" y="${-5*flipper_wheel_slope*scale-flipper_wheel_bias*scale}" z="${3.4*scale-10*small_wheel_radius*scale}"
-                 roll="0" pitch="${PI*0.5}" yaw="${PI}"
-                 radius="${small_wheel_radius}" wheel_length="${wheel_length}" mass="${small_wheel_mass}" parent="left_rear_flipper"/>
-    <!-- <xacro:link_macro name_link="cronstein" x="0" y="0" z="0" mesh_name="cronstain3.dae" mass="0.477" material="red"
-                      scale="1" ixx="1" ixy="0.0" ixz="0.0" iyy="1" iyz="0.000" izz="1"/>
-    <xacro:joint_macro joint_name="joint_cronstein" type="continuous" parent="base_link" child="cronstein"
-      x="0" y="-1.75" z="0.4" roll="0" pitch="${PI*0.0}" yaw="${PI*0.0}" axis="0 0 1"/>
-    <xacro:link_macro name_link="first_part" x="0" y="0" z="0" mesh_name="first_part_of_arm.dae" mass="2.231"
-                      material="red"
-                      scale="0.01" ixx="1" ixy="0.0" ixz="0.0" iyy="1" iyz="0.000" izz="1"/>
-    <xacro:joint_macro joint_name="joint_first_part" type="continuous" parent="cronstein" child="first_part"
-                       x="0.3" y="0.7" z="0.5" roll="${PI*0.5}" pitch="${PI}" yaw="${PI}" axis="1 0 0"/>
-    <xacro:link_macro name_link="second_part" x="0" y="0" z="0" mesh_name="second_part_of_arm.dae" mass="1.407"
-                      material="red"
-                      scale="0.01" ixx="1" ixy="0.0" ixz="0.0" iyy="1" iyz="0.000" izz="1"/>
-    <xacro:joint_macro joint_name="joint_second_part" type="continuous" parent="first_part" child="second_part"
-                       x="-0.7" y="0" z="3" roll="0" pitch="0" yaw="0" axis="1 0 0"/>
-    <xacro:link_macro name_link="head" x="0" y="0" z="0" mesh_name="head.dae" mass="4.738" material="red"
-                      scale="0.01" ixx="1" ixy="0.0" ixz="0.0" iyy="1" iyz="0.000" izz="1"/>
-    <xacro:joint_macro joint_name="joint_head" type="continuous" parent="second_part" child="head"
-                       x="0.2" y="0" z="-4.2" roll="${PI}" pitch="${PI*0}" yaw="0" axis="1 0 0"/> -->
-   <joint name="imu_joint" type="fixed">
+        <xacro:joint_macro joint_name="joint_${loc}_flipper" type="continuous" parent="base_link"
+                            child="${loc}_flipper"
+                            x="${jx}" y="${jy}" z="${jz}"
+                            roll="${roll}" pitch="${pitch}" yaw="${yaw}" axis="0 -1 0" />
+        <xacro:wheel name_link="${loc}_flipper_wheel" mesh_name="right_flipper_tire.stl" material="grey"
+                 x="${(flipper_length-flipper_wheel_radius-flipper_height/2)*scale}"
+                 y="${-1*flipper_width*scale}" z="${0.01*scale-flipper_height/2}"
+                 roll="0" pitch="0" yaw="0" direction="${direction}"
+                 radius="${flipper_wheel_radius}" wheel_length="${flipper_wheel_length}" mass="${small_wheel_mass}" parent="${loc}_flipper"/>
+        <xacro:macro name="right_flipper_middle_wheel"
+             params="loc index direction">
+            <xacro:wheel name_link="${loc}_flipper_middle_wheel_${index}" mesh_name="right_flipper_tire.stl" material="grey"
+                 x="${(flipper_length-flipper_wheel_radius-index*flipper_wheel_distance-flipper_height/2)*scale}"
+                 y="${-1*flipper_width*scale}"
+                 z="${0.01*scale-flipper_height/2}"
+                 roll="0" pitch="0" yaw="0" direction="${direction}"
+                 radius="${flipper_wheel_radius}" wheel_length="${flipper_wheel_length}" mass="${small_wheel_mass}" parent="${loc}_flipper"/>
+        </xacro:macro>
+        <xacro:right_flipper_middle_wheel loc="${loc}" index="1" direction="${direction}"/>
+        <xacro:right_flipper_middle_wheel loc="${loc}" index="2" direction="${direction}"/>
+        <xacro:right_flipper_middle_wheel loc="${loc}" index="3" direction="${direction}"/>
+        <xacro:right_flipper_middle_wheel loc="${loc}" index="4" direction="${direction}"/>
+    </xacro:macro>
+    <xacro:right_flipper_asm loc="right_front"
+        jx="${(gear_length/2-flipper_height/2-0.02)*scale}"
+        jy="${-1*(base_width/2+gear_width-flipper_width)*scale}"
+        jz="${flipper_height/2}"
+        roll="0" pitch="0" yaw="0"/>
+    <xacro:right_flipper_asm loc="left_rear"
+        jx="${(-1)*(gear_length/2-flipper_height/2-0.02)*scale}"
+        jy="${(base_width/2+gear_width-flipper_width)*scale}"
+        jz="${flipper_height/2}"
+        direction="-1"
+        roll="0" pitch="0" yaw="${PI}"/>
+    <!-- left flipper -->
+    <xacro:macro name="left_flipper_asm" params="loc jx jy jz roll pitch yaw direction:=1">
+        <xacro:link_macro name_link="${loc}_flipper" x="0" y="0" z="0" roll="0" pitch="0" yaw="0" mesh_name="left_front_flipper.stl" mass="${flipper_mass}" material="grey"
+                          scale="${scale}" ixx="1" ixy="0.0" ixz="0.0" iyy="1" iyz="0.000" izz="1"/>
+        <xacro:joint_macro joint_name="joint_${loc}_flipper" type="continuous" parent="base_link" child="${loc}_flipper"
+                            x="${jx}" y="${jy}" z="${jz}" roll="${roll}" pitch="${pitch}" yaw="${yaw}" axis="0 -1 0"/>
+        <xacro:wheel name_link="${loc}_flipper_wheel"  mesh_name="left_flipper_tire.stl" material="grey"
+                     x="${(flipper_length-flipper_wheel_radius-flipper_height/2)*scale}"
+                     y="${flipper_width*scale}"
+                     z="${0.01*scale-flipper_height/2}"
+                     roll="0" pitch="0" yaw="0" direction="${direction}"
+                     radius="${flipper_wheel_radius}" wheel_length="${flipper_wheel_length}" mass="${small_wheel_mass}" parent="${loc}_flipper"/>
+        <xacro:macro name="left_flipper_middle_wheel"
+             params="loc index direction">
+            <xacro:wheel name_link="${loc}_flipper_middle_wheel_${index}" mesh_name="left_flipper_tire.stl" material="grey"
+                     x="${(flipper_length-flipper_wheel_radius-index*flipper_wheel_distance-flipper_height/2)*scale}"
+                     y="${flipper_width*scale}"
+                     z="${0.01*scale-flipper_height/2}"
+                     roll="0" pitch="0" yaw="0" direction="${direction}"
+                     radius="${flipper_wheel_radius}" wheel_length="${flipper_wheel_length}" mass="${small_wheel_mass}" parent="${loc}_flipper"/>
+        </xacro:macro>
+        <xacro:left_flipper_middle_wheel loc="${loc}" index="1" direction="${direction}"/>
+        <xacro:left_flipper_middle_wheel loc="${loc}" index="2" direction="${direction}"/>
+        <xacro:left_flipper_middle_wheel loc="${loc}" index="3" direction="${direction}"/>
+        <xacro:left_flipper_middle_wheel loc="${loc}" index="4" direction="${direction}"/>
+    </xacro:macro>
+    <xacro:left_flipper_asm loc="left_front"
+        jx="${(gear_length/2-flipper_height/2-0.02)*scale}"
+        jy="${(base_width/2+gear_width-flipper_width)*scale}"
+        jz="${flipper_height/2}"
+        roll="0" pitch="0" yaw="0"/>
+    <xacro:left_flipper_asm loc="right_rear"
+        jx="${(-1)*(gear_length/2-flipper_height/2-0.02)*scale}"
+        jy="${(-1)*(base_width/2+gear_width-flipper_width)*scale}"
+        jz="${flipper_height/2}"
+        direction="-1"
+        roll="0" pitch="0" yaw="${PI}"/>
+   <!--<joint name="imu_joint" type="fixed">
        <origin xyz="0 0 0"/>
        <parent link="base_link"/>
@@ -311,5 +250,5 @@
        </geometry>
      </collision>
-   </link>
+   </link>-->
    <!--
    <sick_lms1xx_mount prefix="base" topic="scan"/>
