Commit message: Update pb_control.yaml, pb_control.launch, and 7 more files... 1) Add the 6th flipper wheel on each flipper 2) Fine-tune the track beside the mainbody 3) Revise the variables in xacro file.

File: alice/alice-ros/pairbot/src/pairbot/pb_description/urdf/pairbot.xacro (robot description, xacro)
@@ -5,25 +5,25 @@
     <xacro:property name="PI" value="3.1415926"/>
     <!-- Square dimensions (width x width) of beams  0.1-->
+    <xacro:property name="base_mass" value="40.0"/> <!--100-->
     <xacro:property name="base_length" value="0.6"/> <!--was 0.397-->
     <xacro:property name="base_width"  value="0.42"/>  <!--was 0.1789-->
     <xacro:property name="base_height" value="0.18"/>
-    <xacro:property name="gear_length" value="0.54"/>
+    <xacro:property name="gear_length" value="0.493"/>
     <xacro:property name="gear_width"  value="0.136"/> <!-- = 0.20-0.064 -->
-    <xacro:property name="gear_height" value="0.16"/>
-    <xacro:property name="big_wheel_radius" value="0.05"/>   <!--was 0.09-->
-    <xacro:property name="big_wheel_length" value="0.028"/>
+    <xacro:property name="gear_height" value="0.15"/>
+    <xacro:property name="big_wheel_mass" value="1"/>
+    <xacro:property name="big_wheel_radius" value="0.04"/>   <!--was 0.09-->
+    <xacro:property name="big_wheel_thickness" value="0.12"/>
+    <xacro:property name="flipper_mass" value="2.5"/> <!--77.5-->
     <xacro:property name="flipper_length" value="0.42"/>
     <xacro:property name="flipper_width" value="0.10"/>
     <xacro:property name="flipper_height" value="0.1578"/>
-    <xacro:property name="flipper_wheel_radius" value="0.03"/>
+    <xacro:property name="flipper_wheel_mass" value="0.2"/>
+    <xacro:property name="flipper_wheel_radius" value="0.025"/>
     <xacro:property name="flipper_wheel_length" value="0.017"/>
-    <xacro:property name="flipper_wheel_distance" value="0.065"/>
+    <xacro:property name="flipper_wheel_distance" value="0.051"/>
     <!-- <xacro:property name="ground_clearance" value="0.02517"/>  old 0.05 0.02517-->
     <xacro:property name="scale" value="1"/>
     <xacro:property name="prefix" value="pairbot"/>
-    <xacro:property name="base_mass" value="40.0"/> <!--100-->
-    <xacro:property name="flipper_mass" value="2.5"/> <!--77.5-->
-    <xacro:property name="big_wheel_mass" value="0.1"/>
-    <xacro:property name="small_wheel_mass" value="0.1"/>
     <xacro:include filename="$(find pb_description)/urdf/pairbot.gazebo"/>
     <xacro:include filename="$(find pb_description)/urdf/materials.xacro"/>
@@ -123,10 +123,20 @@
         <xacro:visual_macro mesh_name="mainbody.stl" x="0" y="0" z="0" roll="0" pitch="0" yaw="0"
                                 material="orange" scale="${scale}"/>
-        <xacro:visual_macro mesh_name="left_gears.stl" x="0" y="${base_width/2}" z="0" roll="0" pitch="0" yaw="0"
+        <xacro:visual_macro mesh_name="left_gears.stl" x="0" y="${base_width/2}" z="0.02" roll="0" pitch="0" yaw="0"
                                 material="grey" scale="${scale}"/>
-        <xacro:visual_macro mesh_name="right_gears.stl" x="0" y="${-1*base_width/2}" z="0" roll="0" pitch="0" yaw="0"
+        <xacro:visual_macro mesh_name="right_gears.stl" x="0" y="${-1*base_width/2}" z="0.02" roll="0" pitch="0" yaw="0"
                                 material="grey" scale="${scale}"/>
         <xacro:collision_macro mesh_name="mainbody.stl" x="0" y="0" z="0" roll="0" pitch="0" yaw="0"
                                    scale="${scale}"/>
+        <!--
+        <collision>
+                <origin xyz="${-base_length} ${base_width/2} ${flipper_height/2-0.005}" rpy="0 0 0"/>
+                <geometry><box size="${base_length} ${gear_width-flipper_width} ${flipper_height/2+0.005}"/></geometry>
+        </collision>
+        <collision>
+                <origin xyz="${-base_length} ${-1*base_width/2} ${flipper_height/2-0.005}" rpy="${PI} 0 0"/>
+                <geometry><box size="${base_length} ${gear_width-flipper_width} ${flipper_height/2+0.005}"/></geometry>
+        </collision>
+        -->
         <xacro:inertial_macro x="0" y="0" z="0"
                                   roll="0" pitch="0" yaw="0" mass="${base_mass}"
@@ -134,21 +144,21 @@
     </link>
     <xacro:wheel name_link="right_front_base_link_wheel" mesh_name="right_tire.stl" material="grey"
-                 x="${(big_wheel_radius*2+0.01)*scale}" y="${-1*base_width/2*scale}" z="${(big_wheel_radius-0.04)*scale}" roll="0" pitch="0" yaw="0"
-                 radius="${big_wheel_radius}" wheel_length="${big_wheel_length}" mass="${big_wheel_mass}" parent="base_link"/>
+                 x="${(big_wheel_radius*2+0.01)*scale}" y="${-1*base_width/2*scale}" z="${(big_wheel_radius-0.02)*scale}" roll="0" pitch="0" yaw="0"
+                 radius="${big_wheel_radius}" wheel_length="${big_wheel_thickness}" mass="${big_wheel_mass}" parent="base_link"/>
     <xacro:wheel name_link="right_middle_base_link_wheel"  mesh_name="right_tire.stl" material="grey"
-                 x="0" y="${-1*base_width/2*scale}" z="${(big_wheel_radius-0.04)*scale}" roll="0" pitch="0" yaw="0"
-                 radius="${big_wheel_radius}" wheel_length="${big_wheel_length}" mass="${big_wheel_mass}" parent="base_link"/>
+                 x="0" y="${-1*base_width/2*scale}" z="${(big_wheel_radius-0.02)*scale}" roll="0" pitch="0" yaw="0"
+                 radius="${big_wheel_radius}" wheel_length="${big_wheel_thickness}" mass="${big_wheel_mass}" parent="base_link"/>
     <xacro:wheel name_link="right_rear_base_link_wheel" mesh_name="right_tire.stl" material="grey"
-                 x="${-1*(big_wheel_radius*2+0.01)*scale}" y="${-1*base_width/2*scale}" z="${(big_wheel_radius-0.04)*scale}" roll="0" pitch="0" yaw="0"
-                 radius="${big_wheel_radius}" wheel_length="${big_wheel_length}" mass="${big_wheel_mass}" parent="base_link"/>
+                 x="${-1*(big_wheel_radius*2+0.01)*scale}" y="${-1*base_width/2*scale}" z="${(big_wheel_radius-0.02)*scale}" roll="0" pitch="0" yaw="0"
+                 radius="${big_wheel_radius}" wheel_length="${big_wheel_thickness}" mass="${big_wheel_mass}" parent="base_link"/>
     <xacro:wheel name_link="left_front_base_link_wheel" mesh_name="left_tire.stl" material="grey"
-                 x="${(big_wheel_radius*2+0.01)*scale}" y="${base_width/2*scale}" z="${(big_wheel_radius-0.04)*scale}" roll="0" pitch="0" yaw="0"
-                 radius="${big_wheel_radius}" wheel_length="${big_wheel_length}" mass="${big_wheel_mass}" parent="base_link"/>
+                 x="${(big_wheel_radius*2+0.01)*scale}" y="${base_width/2*scale}" z="${(big_wheel_radius-0.02)*scale}" roll="0" pitch="0" yaw="0"
+                 radius="${big_wheel_radius}" wheel_length="${big_wheel_thickness}" mass="${big_wheel_mass}" parent="base_link"/>
     <xacro:wheel name_link="left_middle_base_link_wheel" mesh_name="left_tire.stl" material="grey"
-                 x="0" y="${base_width/2*scale}" z="${(big_wheel_radius-0.04)*scale}" roll="0" pitch="0" yaw="0"
-                radius="${big_wheel_radius}" wheel_length="${big_wheel_length}" mass="${big_wheel_mass}" parent="base_link"/>
+                 x="0" y="${base_width/2*scale}" z="${(big_wheel_radius-0.02)*scale}" roll="0" pitch="0" yaw="0"
+                radius="${big_wheel_radius}" wheel_length="${big_wheel_thickness}" mass="${big_wheel_mass}" parent="base_link"/>
     <xacro:wheel name_link="left_rear_base_link_wheel" mesh_name="left_tire.stl" material="grey"
-                 x="${-1*(big_wheel_radius*2+0.01)*scale}" y="${base_width/2*scale}" z="${(big_wheel_radius-0.04)*scale}" roll="0" pitch="0" yaw="0"
-                 radius="${big_wheel_radius}" wheel_length="${big_wheel_length}" mass="${big_wheel_mass}" parent="base_link"/>
+                 x="${-1*(big_wheel_radius*2+0.01)*scale}" y="${base_width/2*scale}" z="${(big_wheel_radius-0.02)*scale}" roll="0" pitch="0" yaw="0"
+                 radius="${big_wheel_radius}" wheel_length="${big_wheel_thickness}" mass="${big_wheel_mass}" parent="base_link"/>
 <!-- y=3.4 x=0.3--> <!--for flipper: x: left/right y: up/down-->
     <xacro:macro name="right_flipper_asm"
@@ -164,5 +174,5 @@
                  y="${-1*flipper_width*scale}" z="${0.01*scale-flipper_height/2}"
                  roll="0" pitch="0" yaw="0" direction="${direction}"
-                 radius="${flipper_wheel_radius}" wheel_length="${flipper_wheel_length}" mass="${small_wheel_mass}" parent="${loc}_flipper"/>
+                 radius="${flipper_wheel_radius}" wheel_length="${flipper_wheel_length}" mass="${flipper_wheel_mass}" parent="${loc}_flipper"/>
         <xacro:macro name="right_flipper_middle_wheel"
              params="loc index direction">
@@ -172,5 +182,5 @@
                  z="${0.01*scale-flipper_height/2}"
                  roll="0" pitch="0" yaw="0" direction="${direction}"
-                 radius="${flipper_wheel_radius}" wheel_length="${flipper_wheel_length}" mass="${small_wheel_mass}" parent="${loc}_flipper"/>
+                 radius="${flipper_wheel_radius}" wheel_length="${flipper_wheel_length}" mass="${flipper_wheel_mass}" parent="${loc}_flipper"/>
         </xacro:macro>
         <xacro:right_flipper_middle_wheel loc="${loc}" index="1" direction="${direction}"/>
@@ -178,12 +188,14 @@
         <xacro:right_flipper_middle_wheel loc="${loc}" index="3" direction="${direction}"/>
         <xacro:right_flipper_middle_wheel loc="${loc}" index="4" direction="${direction}"/>
+        <xacro:right_flipper_middle_wheel loc="${loc}" index="5" direction="${direction}"/>
+        <xacro:right_flipper_middle_wheel loc="${loc}" index="6" direction="${direction}"/>
     </xacro:macro>
     <xacro:right_flipper_asm loc="right_front"
-        jx="${(gear_length/2-flipper_height/2-0.02)*scale}"
+        jx="${(gear_length/2-flipper_height/2)*scale}"
         jy="${-1*(base_width/2+gear_width-flipper_width)*scale}"
         jz="${flipper_height/2}"
         roll="0" pitch="0" yaw="0"/>
     <xacro:right_flipper_asm loc="left_rear"
-        jx="${(-1)*(gear_length/2-flipper_height/2-0.02)*scale}"
+        jx="${(-1)*(gear_length/2-flipper_height/2)*scale}"
         jy="${(base_width/2+gear_width-flipper_width)*scale}"
         jz="${flipper_height/2}"
@@ -201,5 +213,5 @@
                      z="${0.01*scale-flipper_height/2}"
                      roll="0" pitch="0" yaw="0" direction="${direction}"
-                     radius="${flipper_wheel_radius}" wheel_length="${flipper_wheel_length}" mass="${small_wheel_mass}" parent="${loc}_flipper"/>
+                     radius="${flipper_wheel_radius}" wheel_length="${flipper_wheel_length}" mass="${flipper_wheel_mass}" parent="${loc}_flipper"/>
         <xacro:macro name="left_flipper_middle_wheel"
              params="loc index direction">
@@ -209,5 +221,5 @@
                      z="${0.01*scale-flipper_height/2}"
                      roll="0" pitch="0" yaw="0" direction="${direction}"
-                     radius="${flipper_wheel_radius}" wheel_length="${flipper_wheel_length}" mass="${small_wheel_mass}" parent="${loc}_flipper"/>
+                     radius="${flipper_wheel_radius}" wheel_length="${flipper_wheel_length}" mass="${flipper_wheel_mass}" parent="${loc}_flipper"/>
         </xacro:macro>
         <xacro:left_flipper_middle_wheel loc="${loc}" index="1" direction="${direction}"/>
@@ -215,12 +227,14 @@
         <xacro:left_flipper_middle_wheel loc="${loc}" index="3" direction="${direction}"/>
         <xacro:left_flipper_middle_wheel loc="${loc}" index="4" direction="${direction}"/>
+        <xacro:left_flipper_middle_wheel loc="${loc}" index="5" direction="${direction}"/>
+        <xacro:left_flipper_middle_wheel loc="${loc}" index="6" direction="${direction}"/>
     </xacro:macro>
     <xacro:left_flipper_asm loc="left_front"
-        jx="${(gear_length/2-flipper_height/2-0.02)*scale}"
+        jx="${(gear_length/2-flipper_height/2)*scale}"
         jy="${(base_width/2+gear_width-flipper_width)*scale}"
         jz="${flipper_height/2}"
         roll="0" pitch="0" yaw="0"/>
     <xacro:left_flipper_asm loc="right_rear"
-        jx="${(-1)*(gear_length/2-flipper_height/2-0.02)*scale}"
+        jx="${(-1)*(gear_length/2-flipper_height/2)*scale}"
         jy="${(-1)*(base_width/2+gear_width-flipper_width)*scale}"
         jz="${flipper_height/2}"

Commit message: Update pb_control.yaml, camera_body.stl, and pairbot.xacro
Add camera_stick and refine the PID of flipper

File: alice/alice-ros/pairbot/src/pairbot/pb_description/urdf/pairbot.xacro (robot description, xacro)
@@ -143,4 +143,12 @@
                                   ixx="1" ixy="0" ixz="0" iyy="1" iyz="0" izz="1"/>
     </link>
+    <xacro:link_macro name_link="camera_stick_link" x="0" y="0" z="0" roll="0" pitch="0" yaw="0" mesh_name="camera_body.stl"  mass="5" material="grey"
+                      scale="${scale}" ixx="1" ixy="0.0" ixz="0.0" iyy="1" iyz="0.000" izz="1"/>
+    <joint name="joint_camera_stick" type="fixed">
+        <parent link="base_link"/>
+        <child link="camera_stick_link"/>
+        <origin xyz="${base_length/2-0.03} 0 ${base_height-0.05}" rpy="0 0 0"/>
+        <axis xyz="0 0 0"/>
+    </joint>
     <xacro:wheel name_link="right_front_base_link_wheel" mesh_name="right_tire.stl" material="grey"
                  x="${(big_wheel_radius*2+0.01)*scale}" y="${-1*base_width/2*scale}" z="${(big_wheel_radius-0.02)*scale}" roll="0" pitch="0" yaw="0"
