Commit message: zed model (urdf format)

File: nano/zed/catkin_ws/src/zed_sim_package/urdf/zed_sim.urdf.xacro (robot description, xacro)
@@ -1,26 +1,28 @@
 <?xml version="1.0" ?>
-<robot name="pairbot" xmlns:xacro="http://www.ros.org/wiki/xacro">
-<xarco:include filename="$(find zed_sim_package)/urdf/zed_sim.gazebo.xacro"/>
+  <robot name="Zed_sim" xmlns:xacro="http://www.ros.org/wiki/xacro">
+  <xacro:include filename="$(find zed_sim_package)/urdf/zed_sim.gazebo"/>
+  <!--link name="world"/>
+  <joint name="fixed" type="fixed ">
+    <parent link="world"/>
+    <child link="zed_sim"/>
+	<origin xyz="0.0 0.0 0.02" rpy="0 0 0"/>
+  </joint-->
   <link name="zed_sim">
-      <pose> 0 0 0 0 0 0 </pose>
-      <inertial>
-        <mass>0.159</mass>
-      </inertial>
-      <collision name="collision">
-        <geometry>
-	  <box>
-	    <size> 0.03 0.175 0.033 </size>
-	  </box>
-	</geometry>
-      </collision>
-      <visual name="visual">
-        <pose>-0.02 -0.0875 -0.0125 1.5707963  0 1.5707963 </pose>
-        <geometry>
-          <mesh>
-            <uri>package://zed_sim_package/mesh/zed_body.stl</uri>
-            <scale> 0.001 0.001 0.001</scale>
-	  </mesh>
-        </geometry>
-      </visual>
+	<inertial>
+	  <mass value="0.159"/>
+	  <inertia ixx="0.4" ixy="0.0" ixz="0.0" iyy="0.4" iyz="0.0" izz="0.2"/>
+	</inertial>
+	<collision>
+	  <origin xyz="0 0 0.0 " rpy="0 0 0 "/>
+	  <geometry>
+		<box size="0.03 0.175 0.033"/>
+	  </geometry>
+	</collision>
+	<visual>
+	  <origin xyz="-0.02 -0.0875 -0.0125 " rpy="1.5707963 0 1.5707963"/>
+	  <geometry>
+	     <mesh filename="package://zed_sim_package/mesh/zed_body.stl" scale="0.001 0.001 0.001"/>
+	  </geometry>
+	</visual>
   </link>
 </robot>
