Commit message: base wheel size multiply two times

File: jaden/jaden-pairbot/src/pairbot/pb_description/urdf/pairbot.xacro (robot description, xacro)
@@ -12,5 +12,5 @@
     <xacro:property name="gear_width"  value="0.136"/> <!-- = 0.20-0.064 -->
     <xacro:property name="gear_height" value="0.15"/>
-    <xacro:property name="base_wheel_mass" value="1"/>
+    <xacro:property name="base_wheel_mass" value="0.8"/>
     <xacro:property name="base_wheel_radius" value="0.025"/>   <!--was 0.09-->
     <xacro:property name="flipper_mass" value="2.5"/> <!--77.5-->
@@ -93,4 +93,37 @@
             <xacro:visual_macro mesh_name="${mesh_name}" x="0" y="0" z="0" roll="0" pitch="0" yaw="0"
                                 material="${material}" scale="${scale}"/>
+            <collision>
+                <origin xyz="0 0 0" rpy="${PI/2} 0 0"/>
+                <geometry>
+                	<cylinder radius="${radius*scale}" length="${0.011*scale}"/>
+                </geometry>
+            </collision>
+            <xacro:inertial_macro x="0" y="0" z="0"
+                                  roll="0" pitch="0" yaw="0" mass="${mass}"
+                                  ixx="1" ixy="0.0" ixz="0.0" iyy="1" iyz="0.0" izz="1"/>
+        </link>
+        <joint name="joint_${name_link}" type="continuous">
+            <parent link="${parent}"/>
+            <child link="${name_link}"/>
+            <origin xyz="${x} ${y} ${z}" rpy="${roll} ${pitch} ${yaw}"/>
+            <axis xyz="0 ${direction} 0"/>
+            <limit velocity="20" effort="100"/>
+        </joint>
+        <transmission name="tran_joint_${name_link}">
+            <type>transmission_interface/SimpleTransmission</type>
+            <joint name="joint_${name_link}">
+                <hardwareInterface>hardware_interface/VelocityJointInterface</hardwareInterface>
+            </joint>
+            <actuator name="motor_joint_${name_link}">
+                <hardwareInterface>hardware_interface/VelocityJointInterface</hardwareInterface>
+                <mechanicalReduction>1</mechanicalReduction>
+            </actuator>
+        </transmission>
+    </xacro:macro>
+    <xacro:macro name="wheeltemp"
+                 params="mesh_name material name_link x y z roll pitch yaw radius wheel_length mass parent direction:=1">
+        <link name="${name_link}">
+            <xacro:visual_macro mesh_name="${mesh_name}" x="0" y="0" z="0" roll="0" pitch="0" yaw="0"
+                                material="${material}" scale="${scale*2}"/>
             <collision>
                 <origin xyz="0 0 0" rpy="${PI/2} 0 0"/>
@@ -159,4 +192,24 @@
         </transmission>
     </xacro:macro>
+    <!-- start##In order to improve the performance, I use simple box instead of mesh -->
+    <xacro:macro name="visual_base_box" params="x y z roll pitch yaw material scale mesh_name">
+        <visual>
+            <origin xyz="${x+0.01} ${y} ${z+0.11}" rpy="${roll} ${pitch} ${yaw}"/>
+            <geometry>
+                <box size="${scale*0.37} ${0.46*scale} ${0.12*scale}"/>
+            </geometry>
+            <material name="${material}"/>-->
+        </visual>
+    </xacro:macro>
+    <xacro:macro name="collision_base_box"
+                 params="mesh_name x y z roll pitch yaw scale:=${scale}">
+        <collision>
+            <origin xyz="${x+0.01} ${y} ${z+0.11}" rpy="${roll} ${pitch} ${yaw}"/>
+            <geometry>
+                <box size="${scale*0.37} ${0.46*scale} ${0.12*scale}"/>
+            </geometry>
+        </collision>
+    </xacro:macro>
+    <!-- end##In order to improve the performance, I use simple box instead of mesh -->
     <link name="base_link">
         <xacro:visual_macro mesh_name="mainbody.stl" x="0" y="0" z="0" roll="0" pitch="0" yaw="0"
@@ -166,5 +219,5 @@
         <xacro:visual_macro mesh_name="right_gears.stl" x="0" y="${-1*base_width/2}" z="0.02" roll="0" pitch="0" yaw="0"
                                 material="grey" scale="${scale}"/>
-        <xacro:collision_macro mesh_name="mainbody.stl" x="0" y="0" z="0" roll="0" pitch="0" yaw="0"
+        <xacro:collision_base_box mesh_name="mainbody.stl" x="0" y="0" z="0" roll="0" pitch="0" yaw="0"
                                    scale="${scale}"/>
         <!--
@@ -191,13 +244,13 @@
     </joint>
     <xacro:macro name="right_base_wheel" params="index">
-      <xacro:wheel name_link="right_base_wheel_${index}" mesh_name="right_flipper_tire.stl" material="grey"
-                 x="${base_length/2-0.001-(index-1)*(2*base_wheel_radius+0.001)}"
+      <xacro:wheeltemp name_link="right_base_wheel_${index}" mesh_name="right_flipper_tire.stl" material="grey"
+                 x="${base_length/2-0.001-0.025-(index-1)*(0.05+0.001-0.0045)}"
                  y="${-1*base_width/2}"
-                 z="${base_wheel_radius-0.02}" roll="0" pitch="0" yaw="0"
-                 radius="${base_wheel_radius}" wheel_length="${gear_width-0.005}"
-                 mass="${base_wheel_mass}"
-                 parent="base_link" />
-    </xacro:macro>
-    <xacro:macro name="left_base_wheel" params="index">
+                 z="${0.05-0.02}" roll="0" pitch="0" yaw="0"
+                 radius="${0.05}" wheel_length="${gear_width-0.005}"
+                 mass="${base_wheel_mass}"
+                 parent="base_link" />
+    </xacro:macro>
+    <!-- <xacro:macro name="left_base_wheel" params="index">
       <xacro:wheel name_link="left_base_wheel_${index}" mesh_name="left_flipper_tire.stl" material="grey"
                  x="${base_length/2-0.001-(index-1)*(2*base_wheel_radius+0.001)}"
@@ -207,15 +260,24 @@
                  mass="${base_wheel_mass}"
                  parent="base_link" />
+    </xacro:macro> -->
+    <xacro:macro name="left_base_wheel" params="index">
+      <xacro:wheeltemp name_link="left_base_wheel_${index}" mesh_name="left_flipper_tire.stl" material="grey"
+                 x="${base_length/2-0.001-0.025-(index-1)*(0.05+0.001-0.0045)}"
+                 y="${base_width/2}"
+                 z="${0.05-0.02}" roll="0" pitch="0" yaw="0"
+                 radius="${0.05}" wheel_length="${gear_width-0.005}"
+                 mass="${base_wheel_mass}"
+                 parent="base_link" />
     </xacro:macro>
     <xacro:macro name="right_base_wheel_2nd" params="index">
-      <xacro:wheel name_link="right_base_wheel_2nd_${index}" mesh_name="right_flipper_tire.stl" material="grey"
-                 x="${base_length/2-0.001-(index-1)*(2*base_wheel_radius+0.001)-base_wheel_radius}"
+      <xacro:wheeltemp name_link="right_base_wheel_2nd_${index}" mesh_name="right_flipper_tire.stl" material="grey"
+                 x="${base_length/2-0.001-0.025-(index-1)*(0.05+0.001-0.0045)-0.025}"
                  y="${-1*base_width/2-0.026}"
-                 z="${base_wheel_radius-0.02}" roll="0" pitch="0" yaw="0"
-                 radius="${base_wheel_radius}" wheel_length="${gear_width-0.005}"
-                 mass="${base_wheel_mass}"
-                 parent="base_link" />
-    </xacro:macro>
-    <xacro:macro name="left_base_wheel_2nd" params="index">
+                 z="${0.05-0.02}" roll="0" pitch="0" yaw="0"
+                 radius="${0.05}" wheel_length="${gear_width-0.005}"
+                 mass="${base_wheel_mass}"
+                 parent="base_link" />
+    </xacro:macro>
+    <!-- <xacro:macro name="left_base_wheel_2nd" params="index">
       <xacro:wheel name_link="left_base_wheel_2nd_${index}" mesh_name="left_flipper_tire.stl" material="grey"
                  x="${base_length/2-0.001-(index-1)*(2*base_wheel_radius+0.001)-base_wheel_radius}"
@@ -223,4 +285,13 @@
                  z="${base_wheel_radius-0.02}" roll="0" pitch="0" yaw="0"
                  radius="${base_wheel_radius}" wheel_length="${gear_width-0.005}"
+                 mass="${base_wheel_mass}"
+                 parent="base_link" />
+    </xacro:macro> -->
+    <xacro:macro name="left_base_wheel_2nd" params="index">
+      <xacro:wheeltemp name_link="left_base_wheel_2nd_${index}" mesh_name="left_flipper_tire.stl" material="grey"
+                 x="${base_length/2-0.001-0.025-(index-1)*(0.05+0.001-0.0045)-0.025}"
+                 y="${base_width/2+0.026}"
+                 z="${0.05-0.02}" roll="0" pitch="0" yaw="0"
+                 radius="${0.05}" wheel_length="${gear_width-0.005}"
                  mass="${base_wheel_mass}"
                  parent="base_link" />
@@ -310,10 +381,10 @@
                  radius="${flipper_wheel_radius}" wheel_length="${flipper_width-0.02}" mass="${flipper_wheel_mass}" parent="${loc}_flipper"/>
         </xacro:macro>
-        <xacro:right_flipper_middle_wheel_2nd loc="${loc}" index="1" direction="${direction}"/>
+        <!-- <xacro:right_flipper_middle_wheel_2nd loc="${loc}" index="1" direction="${direction}"/>
         <xacro:right_flipper_middle_wheel_2nd loc="${loc}" index="2" direction="${direction}"/>
         <xacro:right_flipper_middle_wheel_2nd loc="${loc}" index="3" direction="${direction}"/>
         <xacro:right_flipper_middle_wheel_2nd loc="${loc}" index="4" direction="${direction}"/>
         <xacro:right_flipper_middle_wheel_2nd loc="${loc}" index="5" direction="${direction}"/>
-        <xacro:right_flipper_middle_wheel_2nd loc="${loc}" index="6" direction="${direction}"/>
+        <xacro:right_flipper_middle_wheel_2nd loc="${loc}" index="6" direction="${direction}"/> -->
     </xacro:macro>
     <xacro:right_flipper_asm loc="right_front"
@@ -364,10 +435,10 @@
                  radius="${flipper_wheel_radius}" wheel_length="${flipper_width-0.02}" mass="${flipper_wheel_mass}" parent="${loc}_flipper"/>
         </xacro:macro>
-        <xacro:left_flipper_middle_wheel_2nd loc="${loc}" index="1" direction="${direction}"/>
+        <!-- <xacro:left_flipper_middle_wheel_2nd loc="${loc}" index="1" direction="${direction}"/>
         <xacro:left_flipper_middle_wheel_2nd loc="${loc}" index="2" direction="${direction}"/>
         <xacro:left_flipper_middle_wheel_2nd loc="${loc}" index="3" direction="${direction}"/>
         <xacro:left_flipper_middle_wheel_2nd loc="${loc}" index="4" direction="${direction}"/>
         <xacro:left_flipper_middle_wheel_2nd loc="${loc}" index="5" direction="${direction}"/>
-        <xacro:left_flipper_middle_wheel_2nd loc="${loc}" index="6" direction="${direction}"/>
+        <xacro:left_flipper_middle_wheel_2nd loc="${loc}" index="6" direction="${direction}"/> -->
     </xacro:macro>
     <xacro:left_flipper_asm loc="left_front"
