Commit message: base wheel size multiply three times flipper wheel size multiply two times deleted all of the 2nd wheels fixed zed_sim.urdf.xacro's bug

File: jaden/jaden-pairbot/src/pairbot/pb_description/urdf/pairbot.xacro (robot description, xacro)
@@ -13,5 +13,5 @@
     <xacro:property name="gear_height" value="0.15"/>
     <xacro:property name="base_wheel_mass" value="0.8"/>
-    <xacro:property name="base_wheel_radius" value="0.025"/>   <!--was 0.09-->
+    <xacro:property name="base_wheel_radius" value="0.075"/>   <!--was 0.09-->
     <xacro:property name="flipper_mass" value="2.5"/> <!--77.5-->
     <xacro:property name="flipper_length" value="0.42"/>
@@ -19,7 +19,7 @@
     <xacro:property name="flipper_height" value="0.1578"/>
     <xacro:property name="flipper_wheel_mass" value="0.2"/>
-    <xacro:property name="flipper_wheel_radius" value="0.025"/>
+    <xacro:property name="flipper_wheel_radius" value="0.05"/>
     <xacro:property name="flipper_wheel_length" value="0.017"/>
-    <xacro:property name="flipper_wheel_distance" value="0.051"/>
+    <xacro:property name="flipper_wheel_distance" value="0.032"/>
     <!-- <xacro:property name="ground_clearance" value="0.02517"/>  old 0.05 0.02517-->
     <xacro:property name="scale" value="1"/>
@@ -92,5 +92,5 @@
         <link name="${name_link}">
             <xacro:visual_macro mesh_name="${mesh_name}" x="0" y="0" z="0" roll="0" pitch="0" yaw="0"
-                                material="${material}" scale="${scale}"/>
+                                material="${material}" scale="${scale*2}"/>
             <collision>
                 <origin xyz="0 0 0" rpy="${PI/2} 0 0"/>
@@ -121,9 +121,9 @@
         </transmission>
     </xacro:macro>
-    <xacro:macro name="wheeltemp"
+    <xacro:macro name="basewheel"
                  params="mesh_name material name_link x y z roll pitch yaw radius wheel_length mass parent direction:=1">
         <link name="${name_link}">
             <xacro:visual_macro mesh_name="${mesh_name}" x="0" y="0" z="0" roll="0" pitch="0" yaw="0"
-                                material="${material}" scale="${scale*2}"/>
+                                material="${material}" scale="${scale*3}"/>
             <collision>
                 <origin xyz="0 0 0" rpy="${PI/2} 0 0"/>
@@ -244,54 +244,18 @@
     </joint>
     <xacro:macro name="right_base_wheel" params="index">
-      <xacro:wheeltemp name_link="right_base_wheel_${index}" mesh_name="right_flipper_tire.stl" material="grey"
-                 x="${base_length/2-0.001-0.025-(index-1)*(0.05+0.001-0.0045)}"
+      <xacro:basewheel name_link="right_base_wheel_${index}" mesh_name="right_flipper_tire.stl" material="grey"
+                 x="${base_length/2-0.001-0.075-(index-1)*(0.042)}"
                  y="${-1*base_width/2}"
-                 z="${0.05-0.02}" roll="0" pitch="0" yaw="0"
-                 radius="${0.05}" wheel_length="${gear_width-0.005}"
-                 mass="${base_wheel_mass}"
-                 parent="base_link" />
-    </xacro:macro>
-    <!-- <xacro:macro name="left_base_wheel" params="index">
-      <xacro:wheel name_link="left_base_wheel_${index}" mesh_name="left_flipper_tire.stl" material="grey"
-                 x="${base_length/2-0.001-(index-1)*(2*base_wheel_radius+0.001)}"
-                 y="${base_width/2}"
                  z="${base_wheel_radius-0.02}" roll="0" pitch="0" yaw="0"
                  radius="${base_wheel_radius}" wheel_length="${gear_width-0.005}"
                  mass="${base_wheel_mass}"
                  parent="base_link" />
-    </xacro:macro> -->
+    </xacro:macro>
     <xacro:macro name="left_base_wheel" params="index">
-      <xacro:wheeltemp name_link="left_base_wheel_${index}" mesh_name="left_flipper_tire.stl" material="grey"
-                 x="${base_length/2-0.001-0.025-(index-1)*(0.05+0.001-0.0045)}"
+      <xacro:basewheel name_link="left_base_wheel_${index}" mesh_name="left_flipper_tire.stl" material="grey"
+                 x="${base_length/2-0.001-0.075-(index-1)*(0.042)}"
                  y="${base_width/2}"
-                 z="${0.05-0.02}" roll="0" pitch="0" yaw="0"
-                 radius="${0.05}" wheel_length="${gear_width-0.005}"
-                 mass="${base_wheel_mass}"
-                 parent="base_link" />
-    </xacro:macro>
-    <xacro:macro name="right_base_wheel_2nd" params="index">
-      <xacro:wheeltemp name_link="right_base_wheel_2nd_${index}" mesh_name="right_flipper_tire.stl" material="grey"
-                 x="${base_length/2-0.001-0.025-(index-1)*(0.05+0.001-0.0045)-0.025}"
-                 y="${-1*base_width/2-0.026}"
-                 z="${0.05-0.02}" roll="0" pitch="0" yaw="0"
-                 radius="${0.05}" wheel_length="${gear_width-0.005}"
-                 mass="${base_wheel_mass}"
-                 parent="base_link" />
-    </xacro:macro>
-    <!-- <xacro:macro name="left_base_wheel_2nd" params="index">
-      <xacro:wheel name_link="left_base_wheel_2nd_${index}" mesh_name="left_flipper_tire.stl" material="grey"
-                 x="${base_length/2-0.001-(index-1)*(2*base_wheel_radius+0.001)-base_wheel_radius}"
-                 y="${base_width/2+0.026}"
                  z="${base_wheel_radius-0.02}" roll="0" pitch="0" yaw="0"
                  radius="${base_wheel_radius}" wheel_length="${gear_width-0.005}"
-                 mass="${base_wheel_mass}"
-                 parent="base_link" />
-    </xacro:macro> -->
-    <xacro:macro name="left_base_wheel_2nd" params="index">
-      <xacro:wheeltemp name_link="left_base_wheel_2nd_${index}" mesh_name="left_flipper_tire.stl" material="grey"
-                 x="${base_length/2-0.001-0.025-(index-1)*(0.05+0.001-0.0045)-0.025}"
-                 y="${base_width/2+0.026}"
-                 z="${0.05-0.02}" roll="0" pitch="0" yaw="0"
-                 radius="${0.05}" wheel_length="${gear_width-0.005}"
                  mass="${base_wheel_mass}"
                  parent="base_link" />
@@ -321,26 +285,4 @@
     <xacro:left_base_wheel index="11" />
     <xacro:left_base_wheel index="12" />
-    <xacro:right_base_wheel_2nd index="1" />
-    <xacro:right_base_wheel_2nd index="2" />
-    <xacro:right_base_wheel_2nd index="3" />
-    <xacro:right_base_wheel_2nd index="4" />
-    <xacro:right_base_wheel_2nd index="5" />
-    <xacro:right_base_wheel_2nd index="6" />
-    <xacro:right_base_wheel_2nd index="7" />
-    <xacro:right_base_wheel_2nd index="8" />
-    <xacro:right_base_wheel_2nd index="9" />
-    <xacro:right_base_wheel_2nd index="10" />
-    <xacro:right_base_wheel_2nd index="11" />
-    <xacro:left_base_wheel_2nd index="1" />
-    <xacro:left_base_wheel_2nd index="2" />
-    <xacro:left_base_wheel_2nd index="3" />
-    <xacro:left_base_wheel_2nd index="4" />
-    <xacro:left_base_wheel_2nd index="5" />
-    <xacro:left_base_wheel_2nd index="6" />
-    <xacro:left_base_wheel_2nd index="7" />
-    <xacro:left_base_wheel_2nd index="8" />
-    <xacro:left_base_wheel_2nd index="9" />
-    <xacro:left_base_wheel_2nd index="10" />
-    <xacro:left_base_wheel_2nd index="11" />
 <!-- y=3.4 x=0.3--> <!--for flipper: x: left/right y: up/down-->
     <xacro:macro name="right_flipper_asm"
@@ -354,5 +296,5 @@
         <xacro:wheel name_link="${loc}_flipper_wheel" mesh_name="right_flipper_tire.stl" material="grey"
                  x="${(flipper_length-flipper_wheel_radius-flipper_height/2)*scale}"
-                 y="-0.02" z="${0.01-flipper_height/2}"
+                 y="-0.02" z="${0.032-flipper_height/2}"
                  roll="0" pitch="0" yaw="0" direction="${direction}"
                  radius="${flipper_wheel_radius}" wheel_length="${flipper_width-0.02}" mass="${flipper_wheel_mass}" parent="${loc}_flipper"/>
@@ -362,5 +304,5 @@
                  x="${(flipper_length-flipper_wheel_radius-index*flipper_wheel_distance-flipper_height/2)*scale}"
                  y="-0.02"
-                 z="${0.01-flipper_height/2}"
+                 z="${0.032-flipper_height/2}"
                  roll="0" pitch="0" yaw="0" direction="${direction}"
                  radius="${flipper_wheel_radius}" wheel_length="${flipper_width-0.02}" mass="${flipper_wheel_mass}" parent="${loc}_flipper"/>
@@ -372,19 +314,6 @@
         <xacro:right_flipper_middle_wheel loc="${loc}" index="5" direction="${direction}"/>
         <xacro:right_flipper_middle_wheel loc="${loc}" index="6" direction="${direction}"/>
-        <xacro:macro name="right_flipper_middle_wheel_2nd"
-             params="loc index direction">
-            <xacro:wheel name_link="${loc}_flipper_middle_wheel_2nd_${index}" mesh_name="right_flipper_tire.stl" material="grey"
-                 x="${(flipper_length-flipper_wheel_radius-(index-0.5)*flipper_wheel_distance-flipper_height/2)*scale}"
-                 y="-0.04"
-                 z="${0.01-flipper_height/2}"
-                 roll="0" pitch="0" yaw="0" direction="${direction}"
-                 radius="${flipper_wheel_radius}" wheel_length="${flipper_width-0.02}" mass="${flipper_wheel_mass}" parent="${loc}_flipper"/>
-        </xacro:macro>
-        <!-- <xacro:right_flipper_middle_wheel_2nd loc="${loc}" index="1" direction="${direction}"/>
-        <xacro:right_flipper_middle_wheel_2nd loc="${loc}" index="2" direction="${direction}"/>
-        <xacro:right_flipper_middle_wheel_2nd loc="${loc}" index="3" direction="${direction}"/>
-        <xacro:right_flipper_middle_wheel_2nd loc="${loc}" index="4" direction="${direction}"/>
-        <xacro:right_flipper_middle_wheel_2nd loc="${loc}" index="5" direction="${direction}"/>
-        <xacro:right_flipper_middle_wheel_2nd loc="${loc}" index="6" direction="${direction}"/> -->
+        <xacro:right_flipper_middle_wheel loc="${loc}" index="7" direction="${direction}"/>
+        <xacro:right_flipper_middle_wheel loc="${loc}" index="8" direction="${direction}"/>
     </xacro:macro>
     <xacro:right_flipper_asm loc="right_front"
@@ -408,5 +337,5 @@
                      x="${(flipper_length-flipper_wheel_radius-flipper_height/2)*scale}"
                      y="0.02"
-                     z="${0.01*scale-flipper_height/2}"
+                     z="${0.032*scale-flipper_height/2}"
                      roll="0" pitch="0" yaw="0" direction="${direction}"
                      radius="${flipper_wheel_radius}" wheel_length="${flipper_width-0.02}" mass="${flipper_wheel_mass}" parent="${loc}_flipper"/>
@@ -416,5 +345,5 @@
                      x="${(flipper_length-flipper_wheel_radius-index*flipper_wheel_distance-flipper_height/2)*scale}"
                      y="0.02"
-                     z="${0.01*scale-flipper_height/2}"
+                     z="${0.032*scale-flipper_height/2}"
                      roll="0" pitch="0" yaw="0" direction="${direction}"
                      radius="${flipper_wheel_radius}" wheel_length="${flipper_width-0.02}" mass="${flipper_wheel_mass}" parent="${loc}_flipper"/>
@@ -426,19 +355,6 @@
         <xacro:left_flipper_middle_wheel loc="${loc}" index="5" direction="${direction}"/>
         <xacro:left_flipper_middle_wheel loc="${loc}" index="6" direction="${direction}"/>
-        <xacro:macro name="left_flipper_middle_wheel_2nd"
-             params="loc index direction">
-            <xacro:wheel name_link="${loc}_flipper_middle_wheel_2nd_${index}" mesh_name="right_flipper_tire.stl" material="grey"
-                 x="${(flipper_length-flipper_wheel_radius-(index-0.5)*flipper_wheel_distance-flipper_height/2)*scale}"
-                 y="0.054"
-                 z="${0.01-flipper_height/2}"
-                 roll="0" pitch="0" yaw="0" direction="${direction}"
-                 radius="${flipper_wheel_radius}" wheel_length="${flipper_width-0.02}" mass="${flipper_wheel_mass}" parent="${loc}_flipper"/>
-        </xacro:macro>
-        <!-- <xacro:left_flipper_middle_wheel_2nd loc="${loc}" index="1" direction="${direction}"/>
-        <xacro:left_flipper_middle_wheel_2nd loc="${loc}" index="2" direction="${direction}"/>
-        <xacro:left_flipper_middle_wheel_2nd loc="${loc}" index="3" direction="${direction}"/>
-        <xacro:left_flipper_middle_wheel_2nd loc="${loc}" index="4" direction="${direction}"/>
-        <xacro:left_flipper_middle_wheel_2nd loc="${loc}" index="5" direction="${direction}"/>
-        <xacro:left_flipper_middle_wheel_2nd loc="${loc}" index="6" direction="${direction}"/> -->
+        <xacro:left_flipper_middle_wheel loc="${loc}" index="7" direction="${direction}"/>
+        <xacro:left_flipper_middle_wheel loc="${loc}" index="8" direction="${direction}"/>
     </xacro:macro>
     <xacro:left_flipper_asm loc="left_front"
@@ -453,37 +369,4 @@
         direction="-1"
         roll="0" pitch="0" yaw="${PI}"/>
-   <!--<joint name="imu_joint" type="fixed">
-       <origin xyz="0 0 0"/>
-       <parent link="base_link"/>
-       <child link="imu_link"/>
-     </joint>
-   <link name="imu_link">
-     <inertial>
-       <mass value="0.001"/>
-       <origin rpy="0 0 0" xyz="0 0 0"/>
-       <inertia ixx="0.0001" ixy="0" ixz="0" iyy="0.000001" iyz="0" izz="0.0001"/>
-     </inertial>
-     <visual>
-       <origin rpy="0 0 0" xyz="0 0 0"/>
-       <geometry>
-         <box size="0.1 0.1 0.1"/>
-       </geometry>
-     </visual>
-     <collision>
-       <origin rpy="0 0 0" xyz="0 0 0"/>
-       <geometry>
-         <box size=".1 .1 .1"/>
-       </geometry>
-     </collision>
-   </link>-->
-   <!--
-   <sick_lms1xx_mount prefix="base" topic="scan"/>
-   <joint name="laser_mount_joint" type="fixed">
-     <origin xyz="0.0 0.0 ${scale*0.3}"
-             rpy="0 0 0" />
-     <parent link="base_link" />
-     <child link="base_laser_mount" />
-   </joint>
-   -->
   <joint name="scan_joint" type="fixed">
     <parent link="camera_stick_link"/>

File: jaden/jaden-pairbot/src/zed_sim_package/urdf/zed_sim.urdf.xacro (robot description, xacro)
@@ -3,22 +3,18 @@
 	<!--<xarco:include filename="$(find zed_sim_package)/urdf/zed_sim.gazebo.xacro"/>-->
   <link name="zed_sim">
-      <pose> 0 0 0 0 0 0 </pose>
+    <pose> 0 0 0 0 0 0 </pose>
       <inertial>
-        <mass>0.159</mass>
+        <mass value="0.159" />
+        <inertia ixx="1.0" ixy="0.0" ixz="0.0" iyy="1.0" iyz="0.0" izz="1.0" />
       </inertial>
       <collision name="collision">
         <geometry>
-	  <box>
-	    <size> 0.03 0.175 0.033 </size>
-	  </box>
-	</geometry>
+	        <box size="0.03 0.175 0.033" />
+	      </geometry>
       </collision>
       <visual name="visual">
         <pose>-0.02 -0.0875 -0.0125 1.5707963  0 1.5707963 </pose>
         <geometry>
-          <mesh>
-            <uri>package://zed_sim_package/mesh/zed_body.stl</uri>
-            <scale> 0.001 0.001 0.001</scale>
-	  </mesh>
+          <mesh filename="package://zed_sim_package/mesh/zed_body.stl" scale="0.001 0.001 0.001" />
         </geometry>
       </visual>

Commit message: integrated stair_climbing, it works

File: jaden/jaden-pairbot/src/pairbot/pb_description/urdf/pairbot.xacro (robot description, xacro)
@@ -369,8 +369,12 @@
         direction="-1"
         roll="0" pitch="0" yaw="${PI}"/>
-  <joint name="scan_joint" type="fixed">
-    <parent link="camera_stick_link"/>
-    <child link="zed_sim"/>
-    <origin xyz="0 0 0.65" rpy="0 0 0"/>
-  </joint>
+    <!-- <joint name="scan_joint" type="fixed">
+        <parent link="camera_stick_link"/>
+        <child link="zed_sim"/>
+        <origin xyz="0 0 0.65" rpy="0 0.17 0"/>
+    </joint> -->
+    <xacro:joint_macro joint_name="scan_joint" type="continuous" parent="camera_stick_link"
+                            child="zed_sim"
+                            x="0" y="0" z="0.24"
+                            roll="0" pitch="0" yaw="0" axis="0 1 0" />
 </robot>

File: jaden/jaden-pairbot/src/zed_sim_package/urdf/zed_sim.gazebo.xacro (robot description, xacro)
@@ -3,4 +3,5 @@
   <gazebo reference="zed_sim">
     <sensor name="depth" type="depth">
+    	<!-- <visualize>true</visualize> -->
         <pose> 0 0 0.0375 0 0 0 </pose>
         <update_rate>20</update_rate>
@@ -8,6 +9,6 @@
           <horizontal_fov>1.5707813</horizontal_fov>
           <image>
-            <width>1280</width>
-            <height>720</height>
+            <width>672</width>
+            <height>376</height>
             <format>R8G8B8</format>
           </image>
@@ -46,6 +47,6 @@
           <horizontal_fov>1.5707813</horizontal_fov>
           <image>
-            <width>1280</width>
-            <height>720</height>
+            <width>672</width>
+            <height>376</height>
             <format>R8G8B8</format>
           </image>
@@ -77,5 +78,5 @@
       </sensor>
       <sensor name="left" type="camera">
-        <visualize>true</visualize>
+        <visualize>false</visualize>
 	<pose> 0.005 0.058 0.004 0 0 0 </pose>
         <update_rate>20</update_rate>
@@ -83,6 +84,6 @@
           <horizontal_fov>1.5707813</horizontal_fov>
           <image>
-            <width>1280</width>
-            <height>720</height>
+            <width>672</width>
+            <height>376</height>
             <format>R8G8B8</format>
           </image>

File: jaden/jaden-pairbot/src/zed_sim_package/urdf/zed_sim.urdf.xacro (robot description, xacro)
@@ -14,7 +14,11 @@
       </collision>
       <visual name="visual">
-        <pose>-0.02 -0.0875 -0.0125 1.5707963  0 1.5707963 </pose>
+        <pose>-0.02 -0.0875 -0.0125 1.5707963 0 1.5707963 </pose>
         <geometry>
-          <mesh filename="package://zed_sim_package/mesh/zed_body.stl" scale="0.001 0.001 0.001" />
+          <mesh>
+            <uri>package://zed_sim_package/mesh/zed_body.stl</uri>
+            <scale> 0.001 0.001 0.001</scale>
+	        </mesh>
+          <!-- <mesh filename="package://zed_sim_package/mesh/zed_body.stl" scale="0.001 0.001 0.001" /> -->
         </geometry>
       </visual>

Commit message: add sonar sensor for down stairs, pb_teleop_sub receives the topics from cpp, moving flipper with thread, Now, it can perform "going up stairs" and "going down stairs".  Changes to be committed: 	modified:   jaden/jaden-pairbot/readme.md 	modified:   jaden/jaden-pairbot/src/pairbot/pb_description/urdf/pairbot.gazebo 	modified:   jaden/jaden-pairbot/src/pairbot/pb_description/urdf/pairbot.xacro 	modified:   jaden/jaden-pairbot/src/pairbot/pb_teleop/scripts/pb_teleop_sub.py 	modified:   jaden/jaden-pairbot/src/stair_climbing/launch/down_stair.launch 	modified:   jaden/jaden-pairbot/src/stair_climbing/launch/stair_mark.launch 	modified:   jaden/jaden-pairbot/src/stair_climbing/src/DownStairMode.cpp 	modified:   jaden/jaden-pairbot/src/stair_climbing/src/DownStairMode.h 	modified:   jaden/jaden-pairbot/src/stair_climbing/src/Stair_Det.cpp 	modified:   jaden/jaden-pairbot/src/stair_climbing/src/StairsDet.cpp 	modified:   jaden/jaden-pairbot/src/stair_climbing/src/StairsDet.h 	modified:   jaden/jaden-pairbot/src/stair_climbing/src/UpStairMode.cpp

File: jaden/jaden-pairbot/src/pairbot/pb_description/urdf/pairbot.xacro (robot description, xacro)
@@ -377,5 +377,23 @@
     <xacro:joint_macro joint_name="scan_joint" type="continuous" parent="camera_stick_link"
                             child="zed_sim"
-                            x="0" y="0" z="0.24"
+                            x="0.01" y="0" z="0.24"
                             roll="0" pitch="0" yaw="0" axis="0 1 0" />
+    <joint name="sonar_joint" type="fixed">
+        <origin xyz="${base_length/2-0.01} 0 ${base_height-0.04}" rpy="0 1.57 0"/>
+        <parent link="base_link"/>
+        <child link="sonar_link"/>
+    </joint>
+    <link name="sonar_link">
+        <inertial>
+            <mass value="0.001"/>
+            <origin xyz="0 0 0.0" rpy="0 0 0 "/>
+            <inertia ixx="0.000000017" ixy="0" ixz="0" iyy="0.000000017" iyz="0" izz="0.000000017"/>
+        </inertial>
+        <visual>
+            <origin xyz="0 0 0.0" rpy="0 0 0"/>
+            <geometry>
+                <box size="0.005 0.03 0.02"/>
+            </geometry>
+        </visual>
+    </link>
 </robot>
